File: rc board/rc board.sch (KiCad schematic (older format))
At the start: 13 parts, among them U1 DRV10983

Commit message: Finiched the driver part, and assigned the IOs to the uC.
Parts:
- added C1, C2, C4: 10uF, Capacitor_SMD:C_0603_1608Metric, symbol Device:C_Small
- added C3: 100nF, Capacitor_SMD:C_0603_1608Metric, symbol Device:C_Small
- added C5: 1uF, Capacitor_SMD:C_0603_1608Metric, symbol Device:C_Small
- added D?: D_Schottky_Small, Diode_SMD:D_SOD-123, symbol Device:D_Schottky_Small
- added F1: 370mA, Fuse:FUSC1607X85N, symbol Device:Polyfuse_Small
- added J1: Throttle_bypass, Connector_PinHeader_2.54mm:PinHeader_1x02_P2.54mm_Vertical, symbol Connector_Generic:Conn_01x02
- added J2: CH3_bypass, Connector_PinHeader_2.54mm:PinHeader_1x02_P2.54mm_Vertical, symbol Connector_Generic:Conn_01x02
- added J3: Steering_bypass, Connector_PinHeader_2.54mm:PinHeader_1x02_P2.54mm_Vertical, symbol Connector_Generic:Conn_01x02
- added J4: Throttle_in, Connector_PinHeader_2.54mm:PinHeader_1x03_P2.54mm_Vertical, symbol Connector_Generic:Conn_01x03
- added J5: Throttle_out, Connector_PinHeader_2.54mm:PinHeader_1x03_P2.54mm_Vertical, symbol Connector_Generic:Conn_01x03
- added J6: CH3_in, Connector_PinHeader_2.54mm:PinHeader_1x03_P2.54mm_Vertical, symbol Connector_Generic:Conn_01x03
- added J7: CH3_out, Connector_PinHeader_2.54mm:PinHeader_1x03_P2.54mm_Vertical, symbol Connector_Generic:Conn_01x03
- added J8: Steering_in, Connector_PinHeader_2.54mm:PinHeader_1x03_P2.54mm_Vertical, symbol Connector_Generic:Conn_01x03
- added J9: Steering_out, Connector_PinHeader_2.54mm:PinHeader_1x03_P2.54mm_Vertical, symbol Connector_Generic:Conn_01x03
- added R10, R7, R8, R9: 10, Resistor_SMD:R_0603_1608Metric, symbol Device:R
- added R? (x6): 10k, Resistor_SMD:R_0603_1608Metric, symbol Device:R
- C6: renamed from C1; value 0.01nF -> 10nF; footprint Capacitor_SMD:C_0402_1005Metric -> Capacitor_SMD:C_0603_1608Metric
- L1: renamed from L?; value L_Core_Ferrite_Small -> 47 uH; footprint (none) -> Inductor_SMD:L_Bourns_SRN6045TA
- R1: renamed from R5; footprint Resistor_SMD:R_0805_2012Metric -> Resistor_SMD:R_0603_1608Metric
- R2: renamed from R6; footprint Resistor_SMD:R_0805_2012Metric -> Resistor_SMD:R_0603_1608Metric
- R5: renamed from R7; footprint Resistor_SMD:R_0805_2012Metric -> Resistor_SMD:R_0603_1608Metric
- R6: renamed from R8; footprint Resistor_SMD:R_0805_2012Metric -> Resistor_SMD:R_0603_1608Metric
- renumbered R9 to R11, R10 to R12
Connections:
- net labels added: +5V, +5V_0, +5V_1, +5V_2, +5V_3, Batt_0, Batt_1, Batt_2, Batt_3, CH3_in, CH3_out, DIR_1, DIR_2, DIR_3, Steering_servo_in, Steering_servo_out, Throttle, Throttle_in, Throttle_out, U_0, U_1, U_2, U_3, V_0, V_1, V_2, V_3, W_0, W_1, W_2, W_3
- wire segments 36 -> 71
- no-connect marks 3 -> 2

Commit message: Removed the 3.3V part, powering the uC from 5V.
Parts:
- removed C1: 10uF, Capacitor_SMD:C_0603_1608Metric, symbol Device:C_Small
- removed D?: D_Schottky_Small, Diode_SMD:D_SOD-123, symbol Device:D_Schottky_Small
- removed R1, R2, R5, R6: 10, Resistor_SMD:R_0603_1608Metric, symbol Device:R
- added C?: 1uF, Capacitor_SMD:C_0603_1608Metric, symbol Device:C_Small
Connections:
- net labels removed: +3.3V_0, +3.3V_1, +3.3V_2, +3.3V_3
- wire segments 71 -> 68
Changed lines of the file:
@@
 Wire Wire Line
 	6200 1400 6200 1450
-$Comp
-L power:+3.3V #PWR02
-U 1 1 5EB83CB4
-P 3150 1700
-F 0 "#PWR02" H 3150 1550 50  0001 C CNN
-F 1 "+3.3V" H 3165 1873 50  0000 C CNN
-F 2 "" H 3150 1700 50  0001 C CNN
-F 3 "" H 3150 1700 50  0001 C CNN
-	1    3150 1700
-	1    0    0    -1
-$EndComp
 Text GLabel 2450 2300 0    50   3State ~ 0
 EN_0
@@
 Wire Wire Line
 	5050 2000 4900 2000
-Text GLabel 6350 1450 1    50   Output ~ 0
-+3.3V_0
-$Comp
-L power:+3.3V #PWR05
-U 1 1 5EB9DEDF
-P 5000 3350
-F 0 "#PWR05" H 5000 3200 50  0001 C CNN
-F 1 "+3.3V" H 5015 3523 50  0000 C CNN
-F 2 "" H 5000 3350 50  0001 C CNN
-F 3 "" H 5000 3350 50  0001 C CNN
-	1    5000 3350
-	1    0    0    -1
-$EndComp
-$Comp
-L Device:R R2
-U 1 1 5EB9EAA4
-P 4850 3700
-F 0 "R2" H 4920 3746 50  0000 L CNN
-F 1 "10" H 4920 3655 50  0000 L CNN
-F 2 "Resistor_SMD:R_0603_1608Metric" V 4780 3700 50  0001 C CNN
-F 3 "https://www.mouser.fr/ProductDetail/Vishay-Dale/CRCW080510R0FKEAC?qs=sGAEpiMZZMtlubZbdhIBIIZe04wfiaJWn%252B71JJ2tnCQ%3D" H 4850 3700 50  0001 C CNN
-	1    4850 3700
-	1    0    0    -1
-$EndComp
-$Comp
-L Device:R R5
-U 1 1 5EB9F2F6
-P 5150 3700
-F 0 "R5" H 5220 3746 50  0000 L CNN
-F 1 "10" H 5220 3655 50  0000 L CNN
-F 2 "Resistor_SMD:R_0603_1608Metric" V 5080 3700 50  0001 C CNN
-F 3 "https://www.mouser.fr/ProductDetail/Vishay-Dale/CRCW080510R0FKEAC?qs=sGAEpiMZZMtlubZbdhIBIIZe04wfiaJWn%252B71JJ2tnCQ%3D" H 5150 3700 50  0001 C CNN
-	1    5150 3700
-	1    0    0    -1
-$EndComp
-$Comp
-L Device:R R1
-U 1 1 5EB9F771
-P 4600 3700
-F 0 "R1" H 4670 3746 50  0000 L CNN
-F 1 "10" H 4670 3655 50  0000 L CNN
-F 2 "Resistor_SMD:R_0603_1608Metric" V 4530 3700 50  0001 C CNN
-F 3 "https://www.mouser.fr/ProductDetail/Vishay-Dale/CRCW080510R0FKEAC?qs=sGAEpiMZZMtlubZbdhIBIIZe04wfiaJWn%252B71JJ2tnCQ%3D" H 4600 3700 50  0001 C CNN
-	1    4600 3700
-	1    0    0    -1
-$EndComp
-$Comp
-L Device:R R6
-U 1 1 5EB9FB54
-P 5400 3700
-F 0 "R6" H 5470 3746 50  0000 L CNN
-F 1 "10" H 5470 3655 50  0000 L CNN
-F 2 "Resistor_SMD:R_0603_1608Metric" V 5330 3700 50  0001 C CNN
-F 3 "https://www.mouser.fr/ProductDetail/Vishay-Dale/CRCW080510R0FKEAC?qs=sGAEpiMZZMtlubZbdhIBIIZe04wfiaJWn%252B71JJ2tnCQ%3D" H 5400 3700 50  0001 C CNN
-	1    5400 3700
-	1    0    0    -1
-$EndComp
-Wire Wire Line
-	4600 3550 4850 3550
-Connection ~ 4850 3550
-Connection ~ 5150 3550
-Wire Wire Line
-	5150 3550 5400 3550
-Text GLabel 4600 3850 3    50   Input ~ 0
-+3.3V_0
-Text GLabel 4850 3850 3    50   Input ~ 0
-+3.3V_1
-Text GLabel 5150 3850 3    50   Input ~ 0
-+3.3V_2
-Text GLabel 5400 3850 3    50   Input ~ 0
-+3.3V_3
 Text GLabel 2450 2500 0    50   3State ~ 0
 EN_1
@@
 Text GLabel 6800 3850 3    50   Input ~ 0
 +5V_3
-$Comp
-L power:GND #PWR07
-U 1 1 5EB9FF4B
-P 5650 3750
-F 0 "#PWR07" H 5650 3500 50  0001 C CNN
-F 1 "GND" H 5655 3577 50  0000 C CNN
-F 2 "" H 5650 3750 50  0001 C CNN
-F 3 "" H 5650 3750 50  0001 C CNN
-	1    5650 3750
-	1    0    0    -1
-$EndComp
-$Comp
-L Device:C_Small C1
-U 1 1 5EBA0893
-P 5650 3650
-F 0 "C1" H 5558 3604 50  0000 R CNN
-F 1 "10uF" H 5558 3695 50  0000 R CNN
-F 2 "Capacitor_SMD:C_0603_1608Metric" H 5688 3500 50  0001 C CNN
-F 3 "https://www.mouser.fr/ProductDetail/Wurth-Elektronik/885012205067?qs=sGAEpiMZZMsh%252B1woXyUXj4jKQI6sNRw63P4glUaj4WU%3D" H 5650 3650 50  0001 C CNN
-	1    5650 3650
-	-1   0    0    1
-$EndComp
-Wire Wire Line
-	5400 3550 5650 3550
-Connection ~ 5400 3550
 $Comp
 L Device:Polyfuse_Small F1
@@
 	1    0    0    -1
 $EndComp
-Wire Wire Line
-	4850 3550 5000 3550
-$Comp
-L Device:D_Schottky_Small D?
-U 1 1 5EC66306
-P 5000 3450
-F 0 "D?" V 4954 3518 50  0000 L CNN
-F 1 "D_Schottky_Small" V 5045 3518 50  0000 L CNN
-F 2 "Diode_SMD:D_SOD-123" V 5000 3450 50  0001 C CNN
-F 3 "https://www.mouser.fr/ProductDetail/Vishay-Semiconductors/BAT54W-HG3-08?qs=sGAEpiMZZMtbRapU8LlZDx2r3HTumQniWWKxY%2FhzXd0HAFhVJGEzKQ%3D%3D" V 5000 3450 50  0001 C CNN
-	1    5000 3450
-	0    1    1    0
-$EndComp
-Connection ~ 5000 3550
-Wire Wire Line
-	5000 3550 5150 3550
+$Comp
+L power:+5V #PWR?
+U 1 1 5EC6B685
+P 3150 1700
+F 0 "#PWR?" H 3150 1550 50  0001 C CNN
+F 1 "+5V" H 3165 1873 50  0000 C CNN
+F 2 "" H 3150 1700 50  0001 C CNN
+F 3 "" H 3150 1700 50  0001 C CNN
+	1    3150 1700
+	1    0    0    -1
+$EndComp
+$Comp
+L Device:C_Small C?
+U 1 1 5EC6F916
+P 6350 1350
+F 0 "C?" V 6121 1350 50  0000 C CNN
+F 1 "1uF" V 6212 1350 50  0000 C CNN
+F 2 "Capacitor_SMD:C_0603_1608Metric" H 6388 1200 50  0001 C CNN
+F 3 "https://www.mouser.fr/ProductDetail/KEMET/C0603C105K7PACTU?qs=sGAEpiMZZMs0AnBnWHyRQN7%2FAA2D2lPPos6U11lU8XXhxOv1ll26bQ%3D%3D" H 6350 1350 50  0001 C CNN
+	1    6350 1350
+	1    0    0    -1
+$EndComp
+$Comp
+L power:GND #PWR?
+U 1 1 5EC7407D
+P 6250 1050
+F 0 "#PWR?" H 6250 800 50  0001 C CNN
+F 1 "GND" H 6255 877 50  0000 C CNN
+F 2 "" H 6250 1050 50  0001 C CNN
+F 3 "" H 6250 1050 50  0001 C CNN
+	1    6250 1050
+	1    0    0    -1
+$EndComp
+Wire Wire Line
+	6250 1050 6350 1050
+Wire Wire Line
+	6350 1050 6350 1250
 $EndSCHEMATC

Commit message: Added schottkyes for automatic battery compatibility, and started component layout.
Parts:
- added C7: 10uF, Capacitor_SMD:C_0603_1608Metric, symbol Device:C_Small
- added D2, D3: MBR2045CTI, Package_TO_SOT_THT:TO-251-3-1EP_Horizontal_TabDown, symbol Device:D_Schottky_x2_KCom_AKA
- added J10: 3S, Connector_JST:JST_XH_B4B-XH-A_1x04_P2.50mm_Vertical, symbol Connector:Conn_01x04_Male
- added J11: 4S, Connector_JST:JST_XH_B5B-XH-A_1x05_P2.50mm_Vertical, symbol Connector:Conn_01x05_Male
- added J12: 5S, Connector_JST:JST_XH_B6B-XH-A_1x06_P2.50mm_Vertical, symbol Connector:Conn_01x06_Male
- added J13: 6S, Connector_JST:JST_XH_B7B-XH-A_1x07_P2.50mm_Vertical, symbol Connector:Conn_01x07_Male
- added J14: Mot_0, Connector_JST:JST_XH_B3B-XH-A_1x03_P2.50mm_Vertical, symbol Connector:Conn_01x03_Male
- J1: value Throttle_bypass -> Bypass
- J2: value CH3_bypass -> Bypass
- J3: value Steering_bypass -> Bypass
- gave numbers to parts that had none: 7
Connections:
- net labels added: Batt_0_sense, Batt_1_sense, Batt_2_sense, Batt_3_sense, Batt_4, Batt_4_sense, Batt_5, Batt_5_sense, DIR, Steering_in, Steering_out
- net labels removed: Steering_servo_in, Steering_servo_out, Throttle
- wire segments 68 -> 118

Commit message: More routing, added the second driver.
Parts:
- added C10, C12, C? (x4): 1uF, Capacitor_SMD:C_0603_1608Metric, symbol Device:C_Small
- added C11, C8, C? (x4): 10uF, Capacitor_SMD:C_0603_1608Metric, symbol Device:C_Small
- added C13, C? (x2): 10nF, Capacitor_SMD:C_0603_1608Metric, symbol Device:C_Small
- added C9, C? (x2): 100nF, Capacitor_SMD:C_0603_1608Metric, symbol Device:C_Small
- added D4, D? (x2): BAW56LT3G, Package_TO_SOT_SMD:SOT-23, symbol Device:D_x2_ACom_KKA
- added J15, J? (x2): Mot_0, Connector_JST:JST_XH_B3B-XH-A_1x03_P2.50mm_Vertical, symbol Connector:Conn_01x03_Male
- added L2, L? (x2): 47 uH, Inductor_SMD:L_Bourns_SRN6045TA, symbol Device:L_Core_Ferrite_Small
- added R15, R16, R? (x4): 10k, Resistor_SMD:R_0603_1608Metric, symbol Device:R
- added U2, U? (x2): DRV10983, Package_SO:HTSSOP-24-1EP_4.4x7.8mm_P0.65mm_EP3.4x7.8mm_Mask2.4x4.68mm_ThermalVias, symbol Driver_Motor:DRV10983
Connections:
- net labels removed: DIR_0, DIR_1, DIR_2, DIR_3
- wire segments 118 -> 263
- no-connect marks 2 -> 8

Commit message: Added and placed the last 2 drivers, added the battery monitoring part.
Parts:
- added R? (x5): 560k, Resistor_SMD:R_0603_1608Metric, symbol Device:R
- added R?: 470k, Resistor_SMD:R_0603_1608Metric, symbol Device:R
- added R?: 330k, Resistor_SMD:R_0603_1608Metric, symbol Device:R
- added R?: 180k, Resistor_SMD:R_0603_1608Metric, symbol Device:R
- added R?: 150k, Resistor_SMD:R_0603_1608Metric, symbol Device:R
- added R?: 100k, Resistor_SMD:R_0603_1608Metric, symbol Device:R
- gave numbers to parts that had none: 24
Connections:
- wire segments 263 -> 264

Commit message: Layed down almost all the components but the capacitors.
Parts:
- J15: value Mot_0 -> Mot_1
- J16: value Mot_0 -> Mot_3
- J17: value Mot_0 -> Mot_2
- gave numbers to parts that had none: 10
Changed lines of the file:
@@
 P 10650 2150
 F 0 "J15" H 10622 2082 50  0000 R CNN
-F 1 "Mot_0" H 10622 2173 50  0000 R CNN
+F 1 "Mot_1" H 10622 2173 50  0000 R CNN
 F 2 "Connector_JST:JST_XH_B3B-XH-A_1x03_P2.50mm_Vertical" H 10650 2150 50  0001 C CNN
 F 3 "~" H 10650 2150 50  0001 C CNN
@@
 P 7450 5100
 F 0 "J16" H 7422 5032 50  0000 R CNN
-F 1 "Mot_0" H 7422 5123 50  0000 R CNN
+F 1 "Mot_3" H 7422 5123 50  0000 R CNN
 F 2 "Connector_JST:JST_XH_B3B-XH-A_1x03_P2.50mm_Vertical" H 7450 5100 50  0001 C CNN
 F 3 "~" H 7450 5100 50  0001 C CNN
@@
 P 10700 5100
 F 0 "J17" H 10672 5032 50  0000 R CNN
-F 1 "Mot_0" H 10672 5123 50  0000 R CNN
+F 1 "Mot_2" H 10672 5123 50  0000 R CNN
 F 2 "Connector_JST:JST_XH_B3B-XH-A_1x03_P2.50mm_Vertical" H 10700 5100 50  0001 C CNN
 F 3 "~" H 10700 5100 50  0001 C CNN
@@
 $EndComp
 $Comp
-L Device:R R?
+L Device:R R26
 U 1 1 5F016835
 P 3400 3350
-F 0 "R?" V 3193 3350 50  0000 C CNN
+F 0 "R26" V 3193 3350 50  0000 C CNN
 F 1 "560k" V 3284 3350 50  0000 C CNN
 F 2 "Resistor_SMD:R_0603_1608Metric" V 3330 3350 50  0001 C CNN
@@
 $EndComp
 $Comp
-L Device:R R?
+L Device:R R25
 U 1 1 5F01824D
 P 3250 5300
-F 0 "R?" V 3043 5300 50  0000 C CNN
+F 0 "R25" V 3043 5300 50  0000 C CNN
 F 1 "470k" V 3134 5300 50  0000 C CNN
 F 2 "Resistor_SMD:R_0603_1608Metric" V 3180 5300 50  0001 C CNN
@@
 $EndComp
 $Comp
-L Device:R R?
+L Device:R R27
 U 1 1 5F02885A
 P 3400 3800
-F 0 "R?" V 3193 3800 50  0000 C CNN
+F 0 "R27" V 3193 3800 50  0000 C CNN
 F 1 "560k" V 3284 3800 50  0000 C CNN
 F 2 "Resistor_SMD:R_0603_1608Metric" V 3330 3800 50  0001 C CNN
@@
 $EndComp
 $Comp
-L Device:R R?
+L Device:R R28
 U 1 1 5F028A59
 P 3400 4250
-F 0 "R?" V 3193 4250 50  0000 C CNN
+F 0 "R28" V 3193 4250 50  0000 C CNN
 F 1 "560k" V 3284 4250 50  0000 C CNN
 F 2 "Resistor_SMD:R_0603_1608Metric" V 3330 4250 50  0001 C CNN
@@
 $EndComp
 $Comp
-L Device:R R?
+L Device:R R29
 U 1 1 5F028BFB
 P 3400 4700
-F 0 "R?" V 3193 4700 50  0000 C CNN
+F 0 "R29" V 3193 4700 50  0000 C CNN
 F 1 "560k" V 3284 4700 50  0000 C CNN
 F 2 "Resistor_SMD:R_0603_1608Metric" V 3330 4700 50  0001 C CNN
@@
 $EndComp
 $Comp
-L Device:R R?
+L Device:R R30
 U 1 1 5F028E1B
 P 3400 5150
-F 0 "R?" V 3193 5150 50  0000 C CNN
+F 0 "R30" V 3193 5150 50  0000 C CNN
 F 1 "560k" V 3284 5150 50  0000 C CNN
 F 2 "Resistor_SMD:R_0603_1608Metric" V 3330 5150 50  0001 C CNN
@@
 $EndComp
 $Comp
-L Device:R R?
+L Device:R R24
 U 1 1 5F02904C
 P 3250 4850
-F 0 "R?" V 3043 4850 50  0000 C CNN
+F 0 "R24" V 3043 4850 50  0000 C CNN
 F 1 "330k" V 3134 4850 50  0000 C CNN
 F 2 "Resistor_SMD:R_0603_1608Metric" V 3180 4850 50  0001 C CNN
@@
 $EndComp
 $Comp
-L Device:R R?
+L Device:R R23
 U 1 1 5F0292C3
 P 3250 4400
-F 0 "R?" V 3043 4400 50  0000 C CNN
+F 0 "R23" V 3043 4400 50  0000 C CNN
 F 1 "180k" V 3134 4400 50  0000 C CNN
 F 2 "Resistor_SMD:R_0603_1608Metric" V 3180 4400 50  0001 C CNN
@@
 $EndComp
 $Comp
-L Device:R R?
+L Device:R R22
 U 1 1 5F07D657
 P 3250 3950
-F 0 "R?" V 3043 3950 50  0000 C CNN
+F 0 "R22" V 3043 3950 50  0000 C CNN
 F 1 "150k" V 3134 3950 50  0000 C CNN
 F 2 "Resistor_SMD:R_0603_1608Metric" V 3180 3950 50  0001 C CNN
@@
 $EndComp
 $Comp
-L Device:R R?
+L Device:R R21
 U 1 1 5F07D9CD
 P 3250 3500
-F 0 "R?" V 3043 3500 50  0000 C CNN
+F 0 "R21" V 3043 3500 50  0000 C CNN
 F 1 "100k" V 3134 3500 50  0000 C CNN
 F 2 "Resistor_SMD:R_0603_1608Metric" V 3180 3500 50  0001 C CNN
@@
 Batt_0
 $Comp
-L power:GND #PWR?
+L power:GND #PWR0122
 U 1 1 5F2D5437
 P 3250 3650
-F 0 "#PWR?" H 3250 3400 50  0001 C CNN
+F 0 "#PWR0122" H 3250 3400 50  0001 C CNN
 F 1 "GND" H 3255 3477 50  0000 C CNN
 F 2 "" H 3250 3650 50  0001 C CNN
@@
 $EndComp
 $Comp
-L power:GND #PWR?
+L power:GND #PWR0123
 U 1 1 5F2D5B6E
 P 3250 4100
-F 0 "#PWR?" H 3250 3850 50  0001 C CNN
+F 0 "#PWR0123" H 3250 3850 50  0001 C CNN
 F 1 "GND" H 3255 3927 50  0000 C CNN
 F 2 "" H 3250 4100 50  0001 C CNN
@@
 $EndComp
 $Comp
-L power:GND #PWR?
+L power:GND #PWR0124
 U 1 1 5F2D5E7B
 P 3250 4550
-F 0 "#PWR?" H 3250 4300 50  0001 C CNN
+F 0 "#PWR0124" H 3250 4300 50  0001 C CNN
 F 1 "GND" H 3255 4377 50  0000 C CNN
 F 2 "" H 3250 4550 50  0001 C CNN
@@
 $EndComp
 $Comp
-L power:GND #PWR?
+L power:GND #PWR0125
 U 1 1 5F2D61A9
 P 3250 5000
-F 0 "#PWR?" H 3250 4750 50  0001 C CNN
+F 0 "#PWR0125" H 3250 4750 50  0001 C CNN
 F 1 "GND" H 3255 4827 50  0000 C CNN
 F 2 "" H 3250 5000 50  0001 C CNN
@@
 $EndComp
 $Comp
-L power:GND #PWR?
+L power:GND #PWR0126
 U 1 1 5F2D64B7
 P 3250 5450
-F 0 "#PWR?" H 3250 5200 50  0001 C CNN
+F 0 "#PWR0126" H 3250 5200 50  0001 C CNN
 F 1 "GND" H 3255 5277 50  0000 C CNN
 F 2 "" H 3250 5450 50  0001 C CNN

Commit message: Added caps (everybody loves caps), and placed all the components.
Parts:
- added C?: 1000uF, Capacitor_THT:CP_Radial_D10.0mm_P5.00mm, symbol Device:CP1_Small
- added C? (x6): 1000uF, Capacitor_THT:CP_Radial_D6.3mm_P2.50mm, symbol Device:CP1_Small
Connections:
- wire segments 264 -> 282

Commit message: Continued the rooting of MOT3, unlarged the traces.
Parts:
- gave numbers to parts that had none: 7
Connections:
- wire segments 282 -> 285
Changed lines of the file:
@@
 Wire Wire Line
 	3100 6600 3100 6800
+Text GLabel 1950 7100 2    50   Output ~ 0
+Batt_4
+Text GLabel 1950 7200 2    50   Output ~ 0
+Batt_3
+Text GLabel 1950 7500 2    50   Output ~ 0
+Batt_0
+Text GLabel 1950 7400 2    50   Output ~ 0
+Batt_1
+Text GLabel 1950 7300 2    50   Output ~ 0
+Batt_2
 Text GLabel 1950 7000 2    50   Output ~ 0
-Batt_4
-Text GLabel 1950 7100 2    50   Output ~ 0
-Batt_3
-Text GLabel 1950 7400 2    50   Output ~ 0
-Batt_0
-Text GLabel 1950 7300 2    50   Output ~ 0
-Batt_1
-Text GLabel 1950 7200 2    50   Output ~ 0
-Batt_2
-Text GLabel 1950 6900 2    50   Output ~ 0
 Batt_5
 $Comp
@@
 	1600 6900 1600 6650
 Wire Wire Line
-	1950 7000 2400 7000
-Wire Wire Line
-	2400 7000 2400 7250
-Wire Wire Line
 	2400 7250 2500 7250
-Wire Wire Line
-	1950 7100 2350 7100
-Wire Wire Line
-	2350 7100 2350 7400
 Wire Wire Line
 	2350 7400 2800 7400
@@
 Wire Wire Line
 	3100 6800 3100 7150
-Wire Wire Line
-	1950 7200 2300 7200
-Wire Wire Line
-	2300 7200 2300 7450
 Wire Wire Line
 	2300 7450 2900 7450
@@
 	3250 5600 3550 5600
 $Comp
-L Device:CP1_Small C?
+L Device:CP1_Small C31
 U 1 1 5F3F659C
 P 1700 7500
-F 0 "C?" H 1791 7546 50  0000 L CNN
+F 0 "C31" H 1791 7546 50  0000 L CNN
 F 1 "1000uF" H 1791 7455 50  0000 L CNN
 F 2 "Capacitor_THT:CP_Radial_D6.3mm_P2.50mm" H 1700 7500 50  0001 C CNN
@@
 $EndComp
 $Comp
-L Device:CP1_Small C?
+L Device:CP1_Small C32
 U 1 1 5F3C2B37
 P 3400 6700
-F 0 "C?" H 3491 6746 50  0000 L CNN
+F 0 "C32" H 3491 6746 50  0000 L CNN
 F 1 "1000uF" H 3491 6655 50  0000 L CNN
 F 2 "Capacitor_THT:CP_Radial_D10.0mm_P5.00mm" H 3400 6700 50  0001 C CNN
@@
 $EndComp
 $Comp
-L power:GND #PWR?
+L power:GND #PWR0127
 U 1 1 5F3C1665
 P 3400 6800
-F 0 "#PWR?" H 3400 6550 50  0001 C CNN
+F 0 "#PWR0127" H 3400 6550 50  0001 C CNN
 F 1 "GND" H 3405 6627 50  0000 C CNN
 F 2 "" H 3400 6800 50  0001 C CNN
@@
 $EndComp
 $Comp
-L power:+BATT #PWR?
+L power:+BATT #PWR0128
 U 1 1 5F3C11A6
 P 3400 6600
-F 0 "#PWR?" H 3400 6450 50  0001 C CNN
+F 0 "#PWR0128" H 3400 6450 50  0001 C CNN
 F 1 "+BATT" H 3415 6773 50  0000 C CNN
 F 2 "" H 3400 6600 50  0001 C CNN
@@
 $EndComp
 $Comp
-L Device:CP1_Small C?
+L Device:CP1_Small C30
 U 1 1 5F48A357
 P 1700 7400
-F 0 "C?" V 1472 7400 50  0000 C CNN
+F 0 "C30" V 1472 7400 50  0000 C CNN
 F 1 "1000uF" V 1563 7400 50  0000 C CNN
 F 2 "Capacitor_THT:CP_Radial_D6.3mm_P2.50mm" H 1700 7400 50  0001 C CNN
@@
 $EndComp
 $Comp
-L Device:CP1_Small C?
+L Device:CP1_Small C29
 U 1 1 5F48ABA5
 P 1700 7300
-F 0 "C?" H 1791 7346 50  0000 L CNN
+F 0 "C29" H 1791 7346 50  0000 L CNN
 F 1 "1000uF" H 1791 7255 50  0000 L CNN
 F 2 "Capacitor_THT:CP_Radial_D6.3mm_P2.50mm" H 1700 7300 50  0001 C CNN
@@
 $EndComp
 $Comp
-L Device:CP1_Small C?
+L Device:CP1_Small C28
 U 1 1 5F4ADE7E
 P 1700 7200
-F 0 "C?" H 1791 7246 50  0000 L CNN
+F 0 "C28" H 1791 7246 50  0000 L CNN
 F 1 "1000uF" H 1791 7155 50  0000 L CNN
 F 2 "Capacitor_THT:CP_Radial_D6.3mm_P2.50mm" H 1700 7200 50  0001 C CNN
@@
 $EndComp
 $Comp
-L Device:CP1_Small C?
+L Device:CP1_Small C27
 U 1 1 5F4AE4AD
 P 1700 7100
-F 0 "C?" H 1791 7146 50  0000 L CNN
+F 0 "C27" H 1791 7146 50  0000 L CNN
 F 1 "1000uF" H 1791 7055 50  0000 L CNN
 F 2 "Capacitor_THT:CP_Radial_D6.3mm_P2.50mm" H 1700 7100 50  0001 C CNN
@@
 $EndComp
 $Comp
-L Device:CP1_Small C?
+L Device:CP1_Small C26
 U 1 1 5F4AEC33
 P 1700 7000
-F 0 "C?" H 1791 7046 50  0000 L CNN
-F 1 "1000uF" H 1791 6955 50  0000 L CNN
+F 0 "C26" V 1472 7000 50  0000 C CNN
+F 1 "1000uF" V 1563 7000 50  0000 C CNN
 F 2 "Capacitor_THT:CP_Radial_D6.3mm_P2.50mm" H 1700 7000 50  0001 C CNN
 F 3 "~" H 1700 7000 50  0001 C CNN
 	1    1700 7000
-	0    -1   -1   0
+	0    1    1    0
 $EndComp
 Connection ~ 1600 7400
@@
 Wire Wire Line
 	1600 6650 2500 6650
+Wire Wire Line
+	2300 7300 2300 7450
+Wire Wire Line
+	2350 7200 2350 7400
+Wire Wire Line
+	2400 7100 2400 7250
+Wire Wire Line
+	1950 7500 1800 7500
+Connection ~ 1800 7500
+Wire Wire Line
+	1950 7400 1800 7400
+Connection ~ 1800 7400
+Wire Wire Line
+	1800 7300 2300 7300
+Connection ~ 1800 7300
+Wire Wire Line
+	1800 7200 2350 7200
+Connection ~ 1800 7200
+Wire Wire Line
+	1800 7100 2400 7100
+Connection ~ 1800 7100
+Wire Wire Line
+	1950 7000 1800 7000
+Connection ~ 1800 7000
 $EndSCHEMATC
